File: full_speed_usb_hub.kicad_sch (KiCad schematic)
At the start: 37 parts, among them J1 USB_A, J2 USB_A, J3 USB_A, J4 USB_A, J5 USB_C_Receptacle_USB2.0_14P, U1 ADUM4160, U3 TLV73333PDBVR

Commit message: update BOM and order PCBA
Parts:
- D2, D3, D4, D5: value D -> D SS34 C8678; footprint Diode_SMD:D_0603_1608Metric -> Diode_SMD:D_SMA
- J1, J2, J3, J4: value USB_A -> USB_A C668591; footprint Connector_USB:USB_A_Receptacle_GCT_USB1046 -> Library:USB_A_Receptacle_C668591
- R10, R11, R12, R9: value R 24 -> R 27
- U2: value ~ -> CH334P
Changed lines of the file:
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@@
 			)
 		)
-		(property "Value" "USB_A"
+		(property "Value" "USB_A C668591"
 			(at 193.04 92.71 0)
 			(effects
@@
 			)
 		)
-		(property "Footprint" "Connector_USB:USB_A_Receptacle_GCT_USB1046"
+		(property "Footprint" "Library:USB_A_Receptacle_C668591"
 			(at 196.85 104.14 0)
 			(effects
@@
 			)
 		)
-		(property "Value" "D"
+		(property "Value" "D SS34 C8678"
 			(at 204.47 93.98 0)
 			(effects
@@
 			)
 		)
-		(property "Footprint" "Diode_SMD:D_0603_1608Metric"
+		(property "Footprint" "Diode_SMD:D_SMA"
 			(at 204.47 97.79 0)
 			(effects
@@
 			)
 		)
-		(property "Value" "USB_A"
+		(property "Value" "USB_A C668591"
 			(at 107.95 92.71 0)
 			(effects
@@
 			)
 		)
-		(property "Footprint" "Connector_USB:USB_A_Receptacle_GCT_USB1046"
+		(property "Footprint" "Library:USB_A_Receptacle_C668591"
 			(at 111.76 104.14 0)
 			(effects
@@
 			)
 		)
-		(property "Value" "R 24"
+		(property "Value" "R 27"
 			(at 133.35 56.388 90)
 			(effects
@@
 			)
 		)
-		(property "Value" "D"
+		(property "Value" "D SS34 C8678"
 			(at 119.38 93.98 0)
 			(effects
@@
 			)
 		)
-		(property "Footprint" "Diode_SMD:D_0603_1608Metric"
+		(property "Footprint" "Diode_SMD:D_SMA"
 			(at 119.38 97.79 0)
 			(effects
@@
 			)
 		)
-		(property "Value" "R 24"
+		(property "Value" "R 27"
 			(at 99.314 55.88 90)
 			(effects
@@
 			)
 		)
-		(property "Value" "USB_A"
+		(property "Value" "USB_A C668591"
 			(at 137.16 92.71 0)
 			(effects
@@
 			)
 		)
-		(property "Footprint" "Connector_USB:USB_A_Receptacle_GCT_USB1046"
+		(property "Footprint" "Library:USB_A_Receptacle_C668591"
 			(at 140.97 104.14 0)
 			(effects
@@
 			)
 		)
-		(property "Value" "D"
+		(property "Value" "D SS34 C8678"
 			(at 148.59 93.98 0)
 			(effects
@@
 			)
 		)
-		(property "Footprint" "Diode_SMD:D_0603_1608Metric"
+		(property "Footprint" "Diode_SMD:D_SMA"
 			(at 148.59 97.79 0)
 			(effects
@@
 			)
 		)
-		(property "Value" "R 24"
+		(property "Value" "R 27"
 			(at 133.35 63.5 90)
 			(effects
@@
 			)
 		)
-		(property "Value" "R 24"
+		(property "Value" "R 27"
 			(at 99.06 62.992 90)
 			(effects
@@
 			)
 		)
-		(property "Value" "~"
+		(property "Value" "CH334P"
 			(at 177.8 72.39 0)
 			(effects
@@
 			)
 		)
-		(property "Value" "D"
+		(property "Value" "D SS34 C8678"
 			(at 176.53 93.98 0)
 			(effects
@@
 			)
 		)
-		(property "Footprint" "Diode_SMD:D_0603_1608Metric"
+		(property "Footprint" "Diode_SMD:D_SMA"
 			(at 176.53 97.79 0)
 			(effects
@@
 			)
 		)
-		(property "Value" "USB_A"
+		(property "Value" "USB_A C668591"
 			(at 165.1 92.71 0)
 			(effects
@@
 			)
 		)
-		(property "Footprint" "Connector_USB:USB_A_Receptacle_GCT_USB1046"
+		(property "Footprint" "Library:USB_A_Receptacle_C668591"
 			(at 168.91 104.14 0)
 			(effects
